Commit message: Now it just forces torque with no base movement

File: src/skyforge_description/urdf/skyforge.urdf (robot description, URDF)
Before this commit: robot three_link_arm_flat, 5 links, 4 joints
Joints:
- joint joint1: limit lower=-1.57 upper=1.57 effort=5 velocity=2 -> lower=-3.14 upper=3.14 effort=100000 velocity=100000
- joint joint2: limit lower=-1.57 upper=1.57 effort=5 velocity=2 -> lower=-1.57 upper=1.57 effort=100000 velocity=100000
- joint joint3: limit lower=-1.57 upper=1.57 effort=5 velocity=2 -> lower=-1.57 upper=1.57 effort=100000 velocity=100000
- joint world_to_base: limit lower=-5.0 upper=5.0 effort=50 velocity=1.0 -> lower=-5.0 upper=5.0 effort=50 velocity=5.0

Commit message: EOD 1/7/26 - Finally works! Had to swap back set_command for the non-optional set_value

File: src/skyforge_description/urdf/skyforge.urdf (robot description, URDF)
Before this commit: robot three_link_arm_flat, 5 links, 4 joints
Joints:
- joint joint1: limit lower=-3.14 upper=3.14 effort=100000 velocity=100000 -> lower=-1.57 upper=1.57 effort=100000 velocity=100000

Commit message: New pose and base configuration

File: src/skyforge_description/urdf/skyforge.urdf (robot description, URDF)
Before this commit: robot three_link_arm_flat, 5 links, 4 joints
Joints:
- joint joint1: limit lower=-1.57 upper=1.57 effort=100000 velocity=100000 -> lower=0 upper=3.14 effort=100000 velocity=100000; origin xyz=0.2 0 0 -> xyz=0 0.2 0
