Commit message: xacro used instead of pure urdf

File: src/skyforge_description/urdf/skyforge.urdf.xacro (robot description, xacro)
@@ -1,4 +1,24 @@
 <?xml version="1.0"?>
-<robot name="three_link_arm_flat">
+<robot name="three_link_arm_flat" xmlns:xacro="http://www.ros.org/wiki/xacro">
+  <!-- MARK: Inertias and masses -->
+  <xacro:property name="inertiaLink1" value="0.186466" />
+  <xacro:property name="inertiaLink2" value="0.186466" />
+  <xacro:property name="inertiaLink3" value="15.4373" />
+  <xacro:property name="massLink1" value="3.07" />
+  <xacro:property name="massLink2" value="3.07" />
+  <xacro:property name="massLink3" value="41.218" />
+  <!-- MARK:  Geometry -->
+  <xacro:property name="COMLink1" value="0.207655" />
+  <xacro:property name="COMLink2" value="0.207655" />
+  <xacro:property name="COMLink3" value="0.966762" />
+  <xacro:property name="lengthLink1" value="0.75" />
+  <xacro:property name="lengthLink2" value="0.75" />
+  <xacro:property name="lengthLink3" value="2" />
+  <xacro:property name="radiusLink1" value="0.015" />
+  <xacro:property name="radiusLink2" value="0.015" />
+  <xacro:property name="radiusLink3" value="0.015" />
+  <!-- Delete the line above this once you make it not a cylinder -->
+  <xacro:property name="heightPayload" value="0.5" />
+  <xacro:property name="depthPayload" value="0.35" />
   <!-- Used to give the base a prismatic connection to the world (fixed except in y direction) -->
   <link name="world"/>
@@ -30,8 +50,8 @@
     <visual>
       <geometry>
-        <cylinder radius="0.05" length="0.6"/>
+        <cylinder radius="${radiusLink1}" length="${lengthLink1}"/>
       </geometry>
       <!-- Rotate cylinder so it lies along X-axis -->
-      <origin xyz="0.3 0 0" rpy="0 1.5708 0"/>
+      <origin xyz="${lengthLink1 / 2} 0 0" rpy="0 1.5708 0"/>
       <material name="red">
         <color rgba="1 0 0 1"/>
@@ -40,12 +60,12 @@
     <collision>
       <geometry>
-        <cylinder radius="0.05" length="0.6"/>
-      </geometry>
-      <origin xyz="0.3 0 0" rpy="0 1.5708 0"/>
-    </collision>
-    <inertial>
-      <origin xyz="0.3 0 0" rpy="0 0 0"/>
-      <mass value="1.0"/>
-      <inertia ixx="0.00125" ixy="0.0" ixz="0.0" iyy="0.0306" iyz="0.0" izz="0.0306"/>
+        <cylinder radius="${radiusLink1}" length="${lengthLink1}"/>
+      </geometry>
+      <origin xyz="${lengthLink1 / 2} 0 0" rpy="0 1.5708 0"/>
+    </collision>
+    <inertial>
+      <origin xyz="${COMLink1} 0 0" rpy="0 0 0"/>
+      <mass value="${massLink1}"/>
+      <inertia ixx="${inertiaLink1}" ixy="0.0" ixz="0.0" iyy="0.0" iyz="0.0" izz="${inertiaLink1}"/>
     </inertial>
   </link>
@@ -54,7 +74,7 @@
     <visual>
       <geometry>
-        <cylinder radius="0.05" length="0.6"/>
-      </geometry>
-      <origin xyz="0.3 0 0" rpy="0 1.5708 0"/>
+        <cylinder radius="${radiusLink2}" length="${lengthLink2}"/>
+      </geometry>
+      <origin xyz="${lengthLink2 / 2} 0 0" rpy="0 1.5708 0"/>
       <material name="green">
         <color rgba="0 1 0 1"/>
@@ -63,12 +83,12 @@
     <collision>
       <geometry>
-        <cylinder radius="0.05" length="0.6"/>
-      </geometry>
-      <origin xyz="0.3 0 0" rpy="0 1.5708 0"/>
-    </collision>
-    <inertial>
-      <origin xyz="0.3 0 0" rpy="0 0 0"/>
-      <mass value="1.0"/>
-      <inertia ixx="0.00125" ixy="0.0" ixz="0.0" iyy="0.0306" iyz="0.0" izz="0.0306"/>
+        <cylinder radius="${radiusLink2}" length="${lengthLink2}"/>
+      </geometry>
+      <origin xyz="${lengthLink2 / 2} 0 0" rpy="0 1.5708 0"/>
+    </collision>
+    <inertial>
+      <origin xyz="${COMLink2} 0 0" rpy="0 0 0"/>
+      <mass value="${massLink2}"/>
+      <inertia ixx="${inertiaLink2}" ixy="0.0" ixz="0.0" iyy="0.0" iyz="0.0" izz="${inertiaLink2}"/>
     </inertial>
   </link>
@@ -77,7 +97,7 @@
     <visual>
       <geometry>
-        <cylinder radius="0.05" length="0.6"/>
-      </geometry>
-      <origin xyz="0.3 0 0" rpy="0 1.5708 0"/>
+        <cylinder radius="${radiusLink3}" length="${lengthLink3}"/>
+      </geometry>
+      <origin xyz="${lengthLink3 / 2} 0 0" rpy="0 1.5708 0"/>
       <material name="blue">
         <color rgba="0 0 1 1"/>
@@ -86,12 +106,12 @@
     <collision>
       <geometry>
-        <cylinder radius="0.05" length="0.6"/>
-      </geometry>
-      <origin xyz="0.3 0 0" rpy="0 1.5708 0"/>
-    </collision>
-    <inertial>
-      <origin xyz="0.3 0 0" rpy="0 0 0"/>
-      <mass value="1.0"/>
-      <inertia ixx="0.00125" ixy="0.0" ixz="0.0" iyy="0.0306" iyz="0.0" izz="0.0306"/>
+        <cylinder radius="${radiusLink3}" length="${lengthLink3}"/>
+      </geometry>
+      <origin xyz="${lengthLink3 / 2} 0 0" rpy="0 1.5708 0"/>
+    </collision>
+    <inertial>
+      <origin xyz="${COMLink3} 0 0" rpy="0 0 0"/>
+      <mass value="${massLink3}"/>
+      <inertia ixx="${inertiaLink3}" ixy="0.0" ixz="0.0" iyy="0.0" iyz="0.0" izz="${inertiaLink3}"/>
     </inertial>
   </link>

Commit message: Robot goes wild

File: src/skyforge_description/urdf/skyforge.urdf.xacro (robot description, xacro)
@@ -21,4 +21,5 @@
   <xacro:property name="heightPayload" value="0.5" />
   <xacro:property name="depthPayload" value="0.35" />
+  <!-- MARK: Links -->
   <!-- Used to give the base a prismatic connection to the world (fixed except in y direction) -->
   <link name="world"/>
@@ -97,7 +98,7 @@
     <visual>
       <geometry>
-        <cylinder radius="${radiusLink3}" length="${lengthLink3}"/>
-      </geometry>
-      <origin xyz="${lengthLink3 / 2} 0 0" rpy="0 1.5708 0"/>
+        <box size="${lengthLink3} ${heightPayload} ${depthPayload}"/>
+      </geometry>
+      <origin xyz="${lengthLink3 / 2} 0 0" rpy="0 0 0"/>
       <material name="blue">
         <color rgba="0 0 1 1"/>
@@ -116,4 +117,5 @@
     </inertial>
   </link>
+  <!-- MARK: Joints -->
   <!-- Prismatic joints -->
   <joint name="world_to_base" type="prismatic">
@@ -131,22 +133,23 @@
     <axis xyz="0 0 1"/>
     <limit effort="100000" velocity="100000" lower="0" upper="3.14"/>
-    <dynamics damping="0.1" friction="0.0"/>
+    <dynamics damping="0.0" friction="0.0"/>
   </joint>
   <joint name="joint2" type="revolute">
     <parent link="link1"/>
     <child link="link2"/>
-    <origin xyz="0.6 0 0"/>
+    <origin xyz="${lengthLink1} 0 0"/>
     <axis xyz="0 0 1"/>
     <limit effort="100000" velocity="100000" lower="-1.57" upper="1.57"/>
-    <dynamics damping="0.1" friction="0.0"/>
+    <dynamics damping="0.0" friction="0.0"/>
   </joint>
   <joint name="joint3" type="revolute">
     <parent link="link2"/>
     <child link="link3"/>
-    <origin xyz="0.6 0 0"/>
+    <origin xyz="${lengthLink2} 0 0"/>
     <axis xyz="0 0 1"/>
-    <limit effort="100000" velocity="100000" lower="-1.57" upper="1.57"/>
-    <dynamics damping="0.1" friction="0.0"/>
-  </joint>
+    <limit effort="100000" velocity="100000" lower="-3.14" upper="1.57"/>
+    <dynamics damping="0.0" friction="0.0"/>
+  </joint>
+  <!-- MARK: ROS 2 Control -->
   <ros2_control name="GazeboSimSystem" type="system">
     <hardware>
@@ -189,5 +192,5 @@
       </command_interface>
      <state_interface name="position">
-        <param name="initial_value">-0.5</param>
+        <param name="initial_value">-0.55</param>
      </state_interface>
      <state_interface name="velocity"/>
@@ -196,4 +199,5 @@
     </joint>
   </ros2_control>
+  <!-- MARK: Gazebo Plugin -->
 <gazebo>
   <plugin filename="/opt/ros/jazzy/lib/libgz_ros2_control-system.so" name="gz_ros2_control::GazeboSimROS2ControlPlugin">

Commit message: More realistic scenario

File: src/skyforge_description/urdf/skyforge.urdf.xacro (robot description, xacro)
@@ -68,5 +68,5 @@
       <origin xyz="${COMLink1} 0 0" rpy="0 0 0"/>
       <mass value="${massLink1}"/>
-      <inertia ixx="${inertiaLink1}" ixy="0.0" ixz="0.0" iyy="0.0" iyz="0.0" izz="${inertiaLink1}"/>
+      <inertia ixx="${inertiaLink1}" ixy="0.0" ixz="0.0" iyy="${inertiaLink1}" iyz="0.0" izz="${inertiaLink1}"/>
     </inertial>
   </link>
@@ -91,5 +91,5 @@
       <origin xyz="${COMLink2} 0 0" rpy="0 0 0"/>
       <mass value="${massLink2}"/>
-      <inertia ixx="${inertiaLink2}" ixy="0.0" ixz="0.0" iyy="0.0" iyz="0.0" izz="${inertiaLink2}"/>
+      <inertia ixx="${inertiaLink2}" ixy="0.0" ixz="0.0" iyy="${inertiaLink2}" iyz="0.0" izz="${inertiaLink2}"/>
     </inertial>
   </link>
@@ -107,5 +107,5 @@
     <collision>
       <geometry>
-        <cylinder radius="${radiusLink3}" length="${lengthLink3}"/>
+        <box size="${lengthLink3} ${heightPayload} ${depthPayload}"/>
       </geometry>
       <origin xyz="${lengthLink3 / 2} 0 0" rpy="0 1.5708 0"/>
@@ -114,5 +114,5 @@
       <origin xyz="${COMLink3} 0 0" rpy="0 0 0"/>
       <mass value="${massLink3}"/>
-      <inertia ixx="${inertiaLink3}" ixy="0.0" ixz="0.0" iyy="0.0" iyz="0.0" izz="${inertiaLink3}"/>
+      <inertia ixx="${inertiaLink3}" ixy="0.0" ixz="0.0" iyy="${inertiaLink3}" iyz="0.0" izz="${inertiaLink3}"/>
     </inertial>
   </link>
@@ -158,7 +158,7 @@
    <joint name="world_to_base">
       <command_interface name="position"/>
+      <!-- <command_interface name="velocity"/> -->
       <state_interface name="position"/>
       <state_interface name="velocity"/>
-      <state_interface name="effort"/>
    </joint>
    <joint name="joint1">

Commit message: No limits

File: src/skyforge_description/urdf/skyforge.urdf.xacro (robot description, xacro)
@@ -124,5 +124,5 @@
     <origin xyz="0 0 0"/>
     <axis xyz="0 1 0"/> <!-- movement along Y -->
-    <limit lower="-5.0" upper="5.0" effort="50" velocity="5.0"/>
+    <limit lower="-5.0" upper="200.0" effort="50" velocity="5.0"/>
   </joint>
   <!-- Revolute joints -->

Commit message: Updated pose and went back to og gains

File: src/skyforge_description/urdf/skyforge.urdf.xacro (robot description, xacro)
@@ -130,7 +130,7 @@
     <parent link="base_link"/>
     <child link="link1"/>
-    <origin xyz="0 0.2 0"/>
+    <origin xyz="-0.288677297 0.0 0"/>
     <axis xyz="0 0 1"/>
-    <limit effort="100000" velocity="100000" lower="0" upper="3.14"/>
+    <limit effort="100000" velocity="100000" lower="0.4" upper="3.57"/>
     <dynamics damping="0.0" friction="0.0"/>
   </joint>
@@ -140,5 +140,5 @@
     <origin xyz="${lengthLink1} 0 0"/>
     <axis xyz="0 0 1"/>
-    <limit effort="100000" velocity="100000" lower="-1.57" upper="1.57"/>
+    <limit effort="100000" velocity="100000" lower="-2.89" upper="0.5"/>
     <dynamics damping="0.0" friction="0.0"/>
   </joint>
@@ -148,5 +148,5 @@
     <origin xyz="${lengthLink2} 0 0"/>
     <axis xyz="0 0 1"/>
-    <limit effort="100000" velocity="100000" lower="-3.14" upper="1.57"/>
+    <limit effort="100000" velocity="100000" lower="-0.6" upper="2.57"/>
     <dynamics damping="0.0" friction="0.0"/>
   </joint>
@@ -168,5 +168,5 @@
       </command_interface>
       <state_interface name="position">
-        <param name="initial_value">1.07079632679</param>
+        <param name="initial_value">1.984107747</param>
       </state_interface>
       <state_interface name="velocity"/>
@@ -180,5 +180,5 @@
       </command_interface>
      <state_interface name="position">
-        <param name="initial_value">1.0</param>
+        <param name="initial_value">-1.318508983</param>
      </state_interface>
      <state_interface name="velocity"/>
@@ -192,5 +192,5 @@
       </command_interface>
      <state_interface name="position">
-        <param name="initial_value">-0.5</param>
+        <param name="initial_value">0.905197563</param>
      </state_interface>
      <state_interface name="velocity"/>
